Commit message: Add a hand keypoint frame to R1 and retarget SOMA hands to it
R1 has no hand body, unlike G1 whose tested ("lafan", "g1") mapping targets
left_rubber_hand_link. The SOMA mapping therefore had to target
left_wrist_roll_link, whose ORIGIN is at the wrist while its collision mesh
extends ~8 cm further out to cover the hand. The retargeter matched the origin,
so the hand geometry ended up displaced by that amount -- into the hip in 412 of
700 clips (59%), up to 8.2 cm deep, including ordinary walking.

Adds left/right_hand_link at each wrist link's own inertial COM (0.068 m out),
to both the MuJoCo XML and the URDF, since the retargeter solves against the XML
while viser renders the URDF. They are massless fixed frames with no geom, so:
nbody 38 -> 40 but nq stays 33, total mass and ngeom are unchanged, and no
collision geometry is added. Existing retargeted .npz outputs remain compatible.

Effect on the two worst hand-into-hip clips:

                              penetration            cost
  walk_forward_normal_004   -0.0789 -> -0.0769   0.2486 -> 0.0982
  sit_on_heels_loop_003     -0.0822 -> -0.0608   1.0859 -> 1.0730

So this is primarily a tracking-accuracy fix: matching the hand centre rather
than the wrist joint more than halves cost on the walking clip. It only partly
relieves the penetration, which points at a genuine proportion limit rather than
a mapping error -- R1's hip is bulkier relative to its arm span than a human's,
so a human's hands-beside-hips pose cannot be reproduced with clearance no
matter which point is matched. Quantified over a larger sample separately.

Only the ("soma", "r1") mapping is switched. ("lafan", "r1") is left pointing at
wrist_roll_link because that pipeline is tested and working, and changing it
would alter results the user relies on; it has the same issue and is worth
revisiting deliberately.

Co-Authored-By: Claude Opus 4.8 <noreply@anthropic.com>

File: src/holosoma_retargeting/holosoma_retargeting/models/r1/r1_26dof.urdf (robot description, URDF)
Before this commit: robot R1, 40 links, 39 joints
Links:
- added link left_hand_link
- added link right_hand_link
Joints:
- added joint left_hand_joint: type fixed, parent left_wrist_roll_link, child left_hand_link, origin xyz=0.068045 -0.001688 0.001392 rpy=0 0 0
- added joint right_hand_joint: type fixed, parent right_wrist_roll_link, child right_hand_link, origin xyz=0.068045 0.001688 0.001392 rpy=0 0 0
